File: eagle/Konnektduino.core.Rev.1.0.sch (EAGLE design)
At the start: 19 parts, among them IC1 ATSAMD21G18A-AU, IC3 TPS70933DBVT

Commit message: board updates
Parts:
- added RI1, RI2: 4k7, resistor:R-EU_R0603
Connections:
- net +3V3: now also RI1.2, RI2.1
- net PA22: now also RI2.2
- net PA23: now also RI1.1
Changed lines of the file:
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@@
 <part name="VD2" library="diode" deviceset="DIODE-SCHOTTKY-" device="0603"/>
 <part name="U$2" library="con-molex-usb" deviceset="MICRO-USB-RECEPTACLE" device="47589-0001"/>
+<part name="RI1" library="resistor" library_urn="urn:adsk.eagle:library:348" deviceset="R-EU_" device="R0603" package3d_urn="urn:adsk.eagle:package:26057/1" value="4k7"/>
+<part name="RI2" library="resistor" library_urn="urn:adsk.eagle:library:348" deviceset="R-EU_" device="R0603" package3d_urn="urn:adsk.eagle:package:26057/1" value="4k7"/>
 </parts>
 <sheets>
@@
 <instance part="VD2" gate="G$1" x="88.9" y="7.62"/>
 <instance part="U$2" gate="G$1" x="256.54" y="43.18" rot="R180"/>
+<instance part="RI1" gate="G$1" x="226.06" y="-17.78" rot="R90"/>
+<instance part="RI2" gate="G$1" x="226.06" y="-30.48" rot="R90"/>
 </instances>
 <busses>
@@
 <label x="101.6" y="15.24" size="1.27" layer="95" xref="yes"/>
 </segment>
+<segment>
+<pinref part="RI2" gate="G$1" pin="1"/>
+<wire x1="226.06" y1="-35.56" x2="226.06" y2="-38.1" width="0.1524" layer="91"/>
+<label x="226.06" y="-38.1" size="1.27" layer="95" rot="R270" xref="yes"/>
+</segment>
+<segment>
+<pinref part="RI1" gate="G$1" pin="2"/>
+<wire x1="226.06" y1="-12.7" x2="226.06" y2="-10.16" width="0.1524" layer="91"/>
+<label x="226.06" y="-10.16" size="1.27" layer="95" rot="R90" xref="yes"/>
+</segment>
 </net>
 <net name="X32IN" class="0">
@@
 <segment>
 <pinref part="IC1" gate="G$1" pin="PA23"/>
-<wire x1="203.2" y1="-22.86" x2="210.82" y2="-22.86" width="0.1524" layer="91"/>
-<label x="210.82" y="-22.86" size="1.27" layer="95" xref="yes"/>
+<wire x1="203.2" y1="-22.86" x2="226.06" y2="-22.86" width="0.1524" layer="91"/>
+<label x="231.14" y="-22.86" size="1.27" layer="95" xref="yes"/>
+<pinref part="RI1" gate="G$1" pin="1"/>
+<junction x="226.06" y="-22.86"/>
+<wire x1="226.06" y1="-22.86" x2="231.14" y2="-22.86" width="0.1524" layer="91"/>
 </segment>
 </net>
@@
 <segment>
 <pinref part="IC1" gate="G$1" pin="PA22"/>
-<wire x1="203.2" y1="-25.4" x2="210.82" y2="-25.4" width="0.1524" layer="91"/>
-<label x="210.82" y="-25.4" size="1.27" layer="95" xref="yes"/>
-</segment>
-</net>
+<wire x1="203.2" y1="-25.4" x2="226.06" y2="-25.4" width="0.1524" layer="91"/>
+<label x="231.14" y="-25.4" size="1.27" layer="95" xref="yes"/>
+<pinref part="RI2" gate="G$1" pin="2"/>
+<junction x="226.06" y="-25.4"/>
+<wire x1="226.06" y1="-25.4" x2="231.14" y2="-25.4" width="0.1524" layer="91"/>
+</segment>
+</net>

Commit message: updates
Parts:
- CLO2: value 15pf -> 15pF
- renumbered IC1 to SAMD, IC3 to VR3V3, U$2 to USBCON
