File: eagle/Konnektduino.core.Rev.1.0.brd (EAGLE design)
At the start: 34.3 x 34.3 mm, 19 parts, among them IC1 ATSAMD21G18A-AU, IC3 TPS70933DBVT

Commit message: board updates
Parts:
- added RI1, RI2: 4k7, resistor:R0603
- moved U$2 2.54 mm to (19.7, 2.54)
- moved VD1 1.27 mm to (7.62, 4.45)
- moved VD2 1.27 mm to (7.62, 1.91)
- moved C2 1.27 mm to (10.2, 10.2)
- moved CS4 1.27 mm to (6.35, 27.9)
- moved CS2 0.90 mm to (20.3, 17.1)
- moved R1 0.90 mm to (22.2, 19.1)
- moved CC1 0.90 mm to (18.4, 15.2)
- moved RR2 0.64 mm to (27.9, 6.99)
- moved CS1 0.63 mm to (6.99, 15.2)
- moved IC3 0.63 mm to (14.0, 10.2)
- moved RR1 0.63 mm to (22.9, 13.3)
- moved CR1 0.63 mm to (24.8, 11.4)
- moved CS3 0.63 mm to (17.8, 27.3)
Connections:
- net +3V3: now also RI1.2, RI2.1
- net PA22: now also RI2.2
- net PA23: now also RI1.1
Routing:
- net +3V3: track 0.00 -> 61.8 mm
- net GND: track 0.00 -> 37.1 mm, vias 1 -> 6
- net PB22: track 0.00 -> 24.1 mm, vias 1 -> 2
- net PB09: track 0.00 -> 22.0 mm
- net PB23: track 0.00 -> 21.7 mm, vias 1 -> 2
- net PB08: track 0.00 -> 20.9 mm
- net PA27: track 0.00 -> 20.8 mm, vias 1 -> 2
- net PA02: track 0.00 -> 19.7 mm, vias 1 -> 2
- net USB-: track 0.00 -> 19.6 mm, vias 0 -> 2
- net PA04: track 0.00 -> 19.5 mm
- net PA28: track 0.00 -> 19.3 mm, vias 1 -> 2
- net USB+: track 0.00 -> 18.9 mm, vias 0 -> 2
- net PA23: track 0.00 -> 18.6 mm
- net NRST: track 0.00 -> 18.3 mm
- net PA03: track 0.00 -> 18.1 mm, vias 1 -> 2
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- added copper zone on layer 1, net +3V3
- added copper zone on layer 1, net GND
Other:
- board text added: "+3V3"
- board text added: "+5V"
- board text added: "GND"
- board text added: "NC"
- board text added: "NRST"
- board text added: "PA13"
- board text added: "SWCLK"
- board text added: "SWDIO"
- board text added: "X"

Commit message: updates
Parts:
- CLO2: value 15pf -> 15pF
- renumbered IC1 to SAMD, IC3 to VR3V3, U$2 to USBCON
Other:
- board text added: "PA02"
- board text added: "PA03"
- board text added: "PA04"
- board text added: "PA05"
- board text added: "PA06"
- board text added: "PA07"
- board text added: "PA08"
- board text added: "PA09"
- board text added: "PA10"
- board text added: "PA11"
- board text added: "PA12"
- board text added: "PA14"
- board text added: "PA15"
- board text added: "PA16"
- board text added: "PA17"
- board text added: "PA18"
- board text added: "PA19"
- board text added: "PA20"
- board text added: "PA21"
- board text added: "PA22"
- board text added: "PA23"
- board text added: "PA27 / NRST"
- board text added: "PA28 / SWCLK"
- board text added: "PB02 / SWDIO"
- board text added: "PB03"
- board text added: "PB08"
- board text added: "PB09"
- board text added: "PB10"
- board text added: "PB11"
- board text added: "PB22"
- board text added: "PB23 / GND"
- board text removed: "X"

Commit message: updates
Other:
- board text added: "(SCL) PA23"
- board text added: "(SDA) PA22"
- board text added: "Konnektduino CORE Rev 1.0 0xCDDC"
- board text added: "PA10 (TX)"
- board text added: "PA11 (RX)"
- board text removed: "PA10"
- board text removed: "PA11"
- board text removed: "PA22"
- board text removed: "PA23"
Changed lines of the file:
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@@
 <setting verticaltext="up"/>
 </settings>
-<grid distance="50" unitdist="mil" unit="inch" style="lines" multiple="1" display="yes" altdistance="0.025" altunitdist="inch" altunit="inch"/>
+<grid distance="50" unitdist="mil" unit="inch" style="lines" multiple="1" display="yes" altdistance="5" altunitdist="mil" altunit="inch"/>
 <layers>
 <layer number="1" name="Top" color="4" fill="1" visible="yes" active="yes"/>
@@
 <text x="30.48" y="1.524" size="0.8128" layer="26" rot="MR0">GND</text>
 <text x="30.48" y="4.064" size="0.8128" layer="26" rot="MR0">NC</text>
-<text x="3.81" y="6.604" size="0.8128" layer="26" rot="MR0" align="bottom-right">PA23</text>
-<text x="3.81" y="9.144" size="0.8128" layer="26" rot="MR0" align="bottom-right">PA22</text>
+<text x="3.81" y="6.604" size="0.8128" layer="26" rot="MR0" align="bottom-right">(SCL) PA23</text>
+<text x="3.81" y="9.144" size="0.8128" layer="26" rot="MR0" align="bottom-right">(SDA) PA22</text>
 <text x="3.81" y="11.684" size="0.8128" layer="26" rot="MR0" align="bottom-right">PA21</text>
 <text x="3.81" y="14.224" size="0.8128" layer="26" rot="MR0" align="bottom-right">PA20</text>
@@
 <text x="27.94" y="11.684" size="0.8128" layer="25" align="bottom-right">GND</text>
 <text x="3.81" y="29.464" size="0.8128" layer="26" rot="MR0" align="bottom-right">PA14</text>
-<text x="11.049" y="30.099" size="0.6096" layer="26" rot="MR0" align="bottom-right">PA11</text>
+<text x="11.049" y="29.21" size="0.6096" layer="26" rot="MR0" align="bottom-right">PA11
+(RX)</text>
 <text x="30.48" y="29.464" size="0.8128" layer="26" rot="MR0">PB08</text>
 <text x="8.509" y="30.099" size="0.6096" layer="26" rot="MR0" align="bottom-right">PB10</text>
-<text x="13.589" y="30.099" size="0.6096" layer="26" rot="MR0" align="bottom-right">PA10</text>
+<text x="13.589" y="29.21" size="0.6096" layer="26" rot="MR0" align="bottom-right">PA10
+(TX)</text>
 <text x="16.129" y="30.099" size="0.6096" layer="26" rot="MR0" align="bottom-right">PA09</text>
 <text x="18.669" y="30.099" size="0.6096" layer="26" rot="MR0" align="bottom-right">PA08</text>
@@
 <text x="8.509" y="27.559" size="0.6096" layer="26" rot="MR0" align="bottom-right">PA12</text>
 <text x="8.509" y="26.289" size="0.6096" layer="26" rot="MR0" align="bottom-right">PA13</text>
+<text x="13.589" y="16.383" size="1.016" layer="26" rot="MR0" align="center">Konnektduino
+CORE
+Rev 1.0
+0xCDDC
+</text>
 </plain>
 <attributes>
@@
 <via x="32.385" y="12.065" extent="1-16" drill="1.4"/>
 <via x="15.24" y="13.97" extent="1-16" drill="0.35"/>
-<wire x1="13.470728125" y1="17.002290625" x2="13.470728125" y2="16.830603125" width="0.1524" layer="1"/>
-<wire x1="13.470728125" y1="16.830603125" x2="13.973325" y2="16.32800625" width="0.1524" layer="1"/>
-<wire x1="13.973325" y1="15.236675" x2="15.24" y2="13.97" width="0.1524" layer="1"/>
-<wire x1="13.973325" y1="16.32800625" x2="13.973325" y2="15.236675" width="0.1524" layer="1"/>
+<wire x1="13.470728125" y1="17.002290625" x2="13.470728125" y2="16.891" width="0.1524" layer="1"/>
+<wire x1="15.24" y1="13.97" x2="13.973325" y2="15.236675" width="0.1524" layer="1"/>
 <wire x1="15.748" y1="13.462" x2="30.988" y2="13.462" width="0.1524" layer="16"/>
 <wire x1="30.988" y1="13.462" x2="32.385" y2="12.065" width="0.1524" layer="16"/>
 <wire x1="15.24" y1="13.97" x2="15.748" y2="13.462" width="0.1524" layer="16"/>
+<wire x1="13.973325" y1="15.236675" x2="13.973325" y2="16.506675" width="0.1524" layer="1"/>
+<wire x1="13.589" y1="16.891" x2="13.470728125" y2="16.891" width="0.1524" layer="1"/>
+<wire x1="13.973325" y1="16.506675" x2="13.589" y2="16.891" width="0.1524" layer="1"/>
 </signal>
 <signal name="PB22">
@@
 </drawing>
 <compatibility>
+<note version="6.3" minversion="6.2.2" severity="warning">
+Since Version 6.2.2 text objects can contain more than one line,
+which will not be processed correctly with this version.
+</note>
 <note version="8.2" severity="warning">
 Since Version 8.2, EAGLE supports online libraries. The ids
