File: eagle/Konnektduino.emptyModule.Rev.1.0.brd (EAGLE design)
At the start: 34.3 x 34.3 mm, 0 parts

Commit message: updates
Other:
- board text added: "(SCL) PA23"
- board text added: "(SDA) PA22"
- board text added: "PA10 (TX)"
- board text added: "PA11 (RX)"
- board text removed: "PA10"
- board text removed: "PA11"
- board text removed: "PA22"
- board text removed: "PA23"
Changed lines of the file:
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@@
 <drawing>
 <settings>
-<setting alwaysvectorfont="no"/>
+<setting alwaysvectorfont="yes"/>
 <setting verticaltext="up"/>
 </settings>
-<grid distance="50" unitdist="mil" unit="mm" style="lines" multiple="1" display="yes" altdistance="0.025" altunitdist="inch" altunit="mm"/>
+<grid distance="50" unitdist="mil" unit="inch" style="lines" multiple="1" display="yes" altdistance="5" altunitdist="mil" altunit="inch"/>
 <layers>
 <layer number="1" name="Top" color="4" fill="1" visible="yes" active="yes"/>
@@
 <text x="30.48" y="1.524" size="0.8128" layer="26" rot="MR0">GND</text>
 <text x="30.48" y="4.064" size="0.8128" layer="26" rot="MR0">NC</text>
-<text x="3.81" y="6.604" size="0.8128" layer="26" rot="MR0" align="bottom-right">PA23</text>
-<text x="3.81" y="9.144" size="0.8128" layer="26" rot="MR0" align="bottom-right">PA22</text>
+<text x="3.81" y="6.604" size="0.8128" layer="26" rot="MR0" align="bottom-right">(SCL) PA23</text>
+<text x="3.81" y="9.144" size="0.8128" layer="26" rot="MR0" align="bottom-right">(SDA) PA22</text>
 <text x="3.81" y="11.684" size="0.8128" layer="26" rot="MR0" align="bottom-right">PA21</text>
 <text x="3.81" y="14.224" size="0.8128" layer="26" rot="MR0" align="bottom-right">PA20</text>
@@
 <text x="30.48" y="11.684" size="0.8128" layer="26" rot="MR0">PB23</text>
 <text x="3.81" y="29.464" size="0.8128" layer="26" rot="MR0" align="bottom-right">PA14</text>
-<text x="11.049" y="30.099" size="0.6096" layer="26" rot="MR0" align="bottom-right">PA11</text>
+<text x="11.049" y="29.21" size="0.6096" layer="26" rot="MR0" align="bottom-right">PA11
+(RX)</text>
 <text x="30.48" y="29.464" size="0.8128" layer="26" rot="MR0">PB08</text>
 <text x="8.509" y="30.099" size="0.6096" layer="26" rot="MR0" align="bottom-right">PB10</text>
-<text x="13.589" y="30.099" size="0.6096" layer="26" rot="MR0" align="bottom-right">PA10</text>
+<text x="13.589" y="29.21" size="0.6096" layer="26" rot="MR0" align="bottom-right">PA10
+(TX)</text>
 <text x="16.129" y="30.099" size="0.6096" layer="26" rot="MR0" align="bottom-right">PA09</text>
 <text x="18.669" y="30.099" size="0.6096" layer="26" rot="MR0" align="bottom-right">PA08</text>
@@
 </drawing>
 <compatibility>
+<note version="6.3" minversion="6.2.2" severity="warning">
+Since Version 6.2.2 text objects can contain more than one line,
+which will not be processed correctly with this version.
+</note>
 <note version="8.2" severity="warning">
 Since Version 8.2, EAGLE supports online libraries. The ids
