File: eagle/Konnektduino.knx.Rev.1.0.brd (EAGLE design)
At the start: 34.3 x 34.3 mm, 0 parts

Commit message: updates
Parts:
- added C1: 47nF, rcl:C0603
- added C10: 10uF, rcl:C0603
- added C2: 4.7nF, rcl:C0603
- added C3, C5, C6: 100nF, rcl:C0603
- added C4: 100uF, rcl:PANASONIC_E
- added C7: 1uF, rcl:C0603
- added D1: SS16T3G, SparkFun:SMA-DIODE_ALT
- added D2: 1SMA40CAT3G, 1SMA40CAT3G:DIONM5226X220N
- added JP5: (no value), pinhead:1X01
- added L1: 220uH, Wuerth_PowerMagnetics:WE-PD2_7850
- added R1: 22R, rcl:R1218
- added R2: 1, rcl:R0603
- added SJ1: (no value), jumper:SJW
- added U$2: KNX_KLEMME, Matthias_1:KNX_KLEMME
- added U$4: NCN5120_KNX_TRANSCEIVER, Matthias_1:QFN40
- added Y2: 16MHz, SparkFun:RESONATOR-SMD
Connections:
- new net +3V3: C10.1, C5.1, C6.1, R2.2, U$4.11, U$4.19, U$4.30, U$4.40
- new net GND: C10.2, C3.2, C4.-, C5.2, C6.2, C7.2, D2.1, SJ1.1, U$2.P-, U$4.1, U$4.14, U$4.18, U$4.2, U$4.23, U$4.24, U$4.25, U$4.26, U$4.29, U$4.31, U$4.33, Y2.2
- new net N$140: C3.1, U$4.5
- new net N$160: C2.2, U$4.8
- new net N$174: SJ1.2, U$4.38
- new net N$203: D1.A, U$2.P+
- new net N$222: L1.2, U$4.17
- new net N$242: L1.1, R2.1, U$4.20
- new net N$39: C1.2, U$4.4
- new net N$40: C7.1, U$4.10
- new net N$7: C1.1, D1.C, D2.2, R1.2, U$4.6
- new net N$8: C2.1, U$4.7
- new net N$9: C4.+, U$4.16, U$4.9
- new net N$999: R1.1, U$4.3
- new net RXD: U$4.27
- new net SAVEB: JP5.1, U$4.36
- new net TXAL1: U$4.35, Y2.3
- new net TXAL2: U$4.34, Y2.1
- new net TXD: U$4.28
Routing:
- net GND: track 0.00 -> 86.3 mm, vias 1 -> 0
- net N$7: track 0.00 -> 24.8 mm
- net +3V3: track 0.00 -> 14.8 mm
- net N$999: track 0.00 -> 13.0 mm, vias 0 -> 2
- net N$9: track 0.00 -> 12.8 mm
- net N$242: track 0.00 -> 11.4 mm
- net N$203: track 0.00 -> 6.91 mm
- net N$8: track 0.00 -> 5.67 mm
- net TXAL1: track 0.00 -> 4.88 mm
- net N$160: track 0.00 -> 3.67 mm
- net N$39: track 0.00 -> 3.45 mm
- net TXAL2: track 0.00 -> 3.43 mm
- net N$40: track 0.00 -> 3.32 mm
- net N$140: track 0.00 -> 2.04 mm, vias 0 -> 1

Commit message: updates
Routing:
- net GND: vias 0 -> 1
- net +3V3: vias 0 -> 1
Changed lines of the file:
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@@
 <setting verticaltext="up"/>
 </settings>
-<grid distance="50" unitdist="mil" unit="inch" style="lines" multiple="1" display="yes" altdistance="5" altunitdist="mil" altunit="inch"/>
+<grid distance="50" unitdist="mil" unit="inch" style="lines" multiple="1" display="yes" altdistance="0.025" altunitdist="inch" altunit="inch"/>
 <layers>
 <layer number="1" name="Top" color="4" fill="1" visible="yes" active="yes"/>
@@
 </elements>
 <signals>
-<signal name="NC01">
-<via x="32.385" y="4.445" extent="1-16" drill="1.4"/>
-<via x="32.385" y="1.905" extent="1-16" drill="1.4"/>
-<wire x1="32.385" y1="1.905" x2="32.385" y2="4.445" width="0" layer="19" extent="1-1"/>
-</signal>
 <signal name="N$1">
 <via x="32.385" y="6.985" extent="1-16" drill="1.4"/>
@@
 <via x="1.905" y="6.985" extent="1-16" drill="1.4"/>
 </signal>
-<signal name="N$37">
-<via x="1.905" y="4.445" extent="1-16" drill="1.4"/>
-</signal>
-<signal name="N$38">
+<signal name="+5V">
 <via x="1.905" y="1.905" extent="1-16" drill="1.4"/>
 </signal>
@@
 <wire x1="12.45" y1="21.2550875" x2="12.633" y2="21.0720875" width="0.3048" layer="1"/>
 <via x="12.633" y="21.0720875" extent="1-16" drill="0.35"/>
-<wire x1="12.633" y1="21.0720875" x2="10.16" y2="18.2" width="0" layer="19" extent="1-1"/>
+<wire x1="10.16" y1="18.2" x2="12.633" y2="21.0720875" width="0" layer="19" extent="1-1"/>
 </signal>
 <signal name="N$39">
@@
 <wire x1="10.45" y1="23.035" x2="10.45" y2="20.19" width="0.3048" layer="1"/>
 <wire x1="10.45" y1="20.19" x2="10.16" y2="19.9" width="0.3048" layer="1"/>
+<via x="32.385" y="1.905" extent="1-16" drill="1.4"/>
+<wire x1="28.4" y1="15.875" x2="32.385" y2="1.905" width="0" layer="19" extent="1-1"/>
 </signal>
 <signal name="N$174">
@@
 <wire x1="18.2" y1="26.035" x2="18.2" y2="27.266" width="0.3048" layer="1"/>
 <wire x1="18.2" y1="27.266" x2="18.161" y2="27.305" width="0.3048" layer="1"/>
+<via x="1.905" y="4.445" extent="1-16" drill="1.4"/>
 <wire x1="15.7" y1="23.785" x2="18.2" y2="26.035" width="0" layer="19" extent="1-1"/>
 <wire x1="10.45" y1="29.035" x2="15.7" y2="27.785" width="0" layer="19" extent="1-1"/>
 <wire x1="9.7" y1="23.785" x2="10.45" y2="29.035" width="0" layer="19" extent="1-1"/>
+<wire x1="1.905" y1="4.445" x2="7.2" y2="21.59" width="0" layer="19" extent="1-1"/>
+</signal>
+<signal name="N$37">
+<via x="32.385" y="4.445" extent="1-16" drill="1.4"/>
 </signal>
 </signals>

Commit message: updates
Parts:
- removed JP5: (no value), pinhead:1X01
- added C11: 10uF, rcl:C0603
- added L2: 220uH, Wuerth_PowerMagnetics:WE-PD2_7850
- added R3: 1, rcl:R0603
- added R4: 33k, rcl:R0603
- added R5: 180k, rcl:R0603
- added VD1, VD2: (no value), diode:D0603
- moved U$2 2.54 mm to (12.7, 2.54)
- renumbered Y2 to Y1
Connections:
- removed net SAVEB: JP5.1, U$4.36
- new net +5V: VD1.C
- new net N$38: L2.2, U$4.15
- new net N$41: R4.2, R5.2, U$4.11
- new net N$42: L2.1, R3.2, U$4.12
- new net VDD1: C10.1, C5.1, C6.1, R2.2, U$4.19, U$4.30, U$4.40, VD2.A
- new net VDD2: C11.1, R3.1, R4.1, U$4.13, VD1.A
- net +3V3: now also VD2.C; no longer C10.1, C5.1, C6.1, R2.2, U$4.11, U$4.19, U$4.30, U$4.40
- net GND: now also C11.2, R5.1
Routing:
- net VDD1: track 0.00 -> 19.4 mm, vias 0 -> 2
- net +3V3: track 14.8 -> 0.00 mm
- net GND: track 86.3 -> 79.3 mm
- net N$203: track 6.91 -> 0.00 mm
Changed lines of the file:
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@@
 <element name="C3" library="rcl" package="C0603" value="100nF" x="10.16" y="19.05" rot="R90"/>
 <element name="C5" library="rcl" package="C0603" value="100nF" x="6.35" y="21.59" rot="R180"/>
-<element name="Y2" library="SparkFun" package="RESONATOR-SMD" value="16MHz" x="6.35" y="25.4" rot="R270"/>
+<element name="Y1" library="SparkFun" package="RESONATOR-SMD" value="16MHz" x="6.35" y="25.4" rot="R270"/>
 <element name="C6" library="rcl" package="C0603" value="100nF" x="6.35" y="29.21" rot="R180"/>
 <element name="C10" library="rcl" package="C0603" value="10uF" x="19.05" y="26.035"/>
 <element name="R2" library="rcl" package="R0603" value="1" x="19.05" y="28.575"/>
 <element name="L1" library="Wuerth_PowerMagnetics" package="WE-PD2_7850" value="220uH" x="25.4" y="25.4" rot="R270"/>
-<element name="U$2" library="Matthias_1" package="KNX_KLEMME" value="KNX_KLEMME" x="10.16" y="2.54" rot="R90"/>
-<element name="JP5" library="pinhead" package="1X01" value="" x="-5.08" y="11.43"/>
+<element name="U$2" library="Matthias_1" package="KNX_KLEMME" value="KNX_KLEMME" x="12.7" y="2.54" rot="R90"/>
 <element name="U$4" library="Matthias_1" package="QFN40" value="NCN5120_KNX_TRANSCEIVER" x="12.7" y="26.035"/>
 <element name="C7" library="rcl" package="C0603" value="1uF" x="19.05" y="22.86"/>
@@
 <element name="C4" library="rcl" package="PANASONIC_E" value="100uF" x="25.4" y="15.875" rot="R180"/>
 <element name="SJ1" library="jumper" library_urn="urn:adsk.eagle:library:252" package="SJW" package3d_urn="urn:adsk.eagle:package:15507/1" value="" x="6.35" y="17.78"/>
+<element name="L2" library="Wuerth_PowerMagnetics" package="WE-PD2_7850" value="220uH" x="25.4" y="6.35" rot="R90"/>
+<element name="R3" library="rcl" package="R0603" value="1" x="18.415" y="9.525"/>
+<element name="C11" library="rcl" package="C0603" value="10uF" x="18.415" y="12.7"/>
+<element name="R4" library="rcl" package="R0603" value="33k" x="19.05" y="19.05" rot="R180"/>
+<element name="R5" library="rcl" package="R0603" value="180k" x="17.78" y="15.875" rot="R180"/>
+<element name="VD1" library="diode" package="D0603" value="" x="18.415" y="6.985"/>
+<element name="VD2" library="diode" package="D0603" value="" x="5.08" y="5.08" rot="R90"/>
 </elements>
 <signals>
@@
 <via x="1.905" y="6.985" extent="1-16" drill="1.4"/>
 </signal>
-<signal name="+5V">
-<via x="1.905" y="1.905" extent="1-16" drill="1.4"/>
+<signal name="VDD2">
+<contactref element="U$4" pad="13"/>
+<contactref element="R3" pad="1"/>
+<contactref element="C11" pad="1"/>
+<contactref element="R4" pad="1"/>
+<contactref element="VD1" pad="A"/>
+<wire x1="19.9" y1="19.05" x2="15.7" y2="24.785" width="0" layer="19" extent="1-1"/>
+<wire x1="17.565" y1="12.7" x2="19.9" y2="19.05" width="0" layer="19" extent="1-1"/>
+<wire x1="17.565" y1="9.525" x2="17.565" y2="12.7" width="0" layer="19" extent="1-1"/>
+<wire x1="19.177" y1="6.985" x2="17.565" y2="9.525" width="0" layer="19" extent="1-1"/>
 </signal>
 <signal name="N$999">
@@
 <contactref element="C6" pad="2"/>
 <contactref element="C5" pad="2"/>
-<contactref element="Y2" pad="2"/>
+<contactref element="Y1" pad="2"/>
 <contactref element="U$4" pad="31"/>
 <contactref element="U$4" pad="33"/>
@@
 <contactref element="C10" pad="2"/>
 <contactref element="SJ1" pad="1"/>
-<wire x1="7.61" y1="2.54" x2="7.61" y2="5.725" width="1.016" layer="1"/>
-<wire x1="7.61" y1="5.725" x2="6.985" y2="6.35" width="1.016" layer="1"/>
-<wire x1="6.985" y1="6.35" x2="6.985" y2="9.28" width="1.016" layer="1"/>
 <wire x1="6.985" y1="9.28" x2="5.08" y2="11.185" width="0.4064" layer="1"/>
 <wire x1="5.08" y1="11.185" x2="5.08" y2="17.78" width="0.4064" layer="1"/>
@@
 <wire x1="10.45" y1="20.19" x2="10.16" y2="19.9" width="0.3048" layer="1"/>
 <via x="32.385" y="1.905" extent="1-16" drill="1.4"/>
-<wire x1="28.4" y1="15.875" x2="32.385" y2="1.905" width="0" layer="19" extent="1-1"/>
+<contactref element="C11" pad="2"/>
+<contactref element="R5" pad="1"/>
+<wire x1="19.265" y1="12.7" x2="18.63" y2="15.875" width="0" layer="19" extent="1-1"/>
+<wire x1="21.463" y1="20.193" x2="18.63" y2="15.875" width="0" layer="19" extent="1-1"/>
+<wire x1="10.15" y1="2.54" x2="6.985" y2="9.28" width="0" layer="19" extent="1-1"/>
+<wire x1="32.385" y1="1.905" x2="28.4" y2="15.875" width="0" layer="19" extent="1-1"/>
 </signal>
 <signal name="N$174">
@@
 <wire x1="7.62" y1="17.78" x2="9.7" y2="24.785" width="0" layer="19" extent="1-1"/>
 </signal>
-<signal name="SAVEB">
-<contactref element="JP5" pad="1"/>
-<contactref element="U$4" pad="36"/>
-<wire x1="-5.08" y1="11.43" x2="9.7" y2="25.785" width="0" layer="19" extent="1-1"/>
-</signal>
 <signal name="TXAL1">
-<contactref element="Y2" pad="3"/>
+<contactref element="Y1" pad="3"/>
 <contactref element="U$4" pad="35"/>
 <wire x1="9.7" y1="26.285" x2="8.251" y2="26.285" width="0.3048" layer="1"/>
@@
 </signal>
 <signal name="TXAL2">
-<contactref element="Y2" pad="1"/>
+<contactref element="Y1" pad="1"/>
 <contactref element="U$4" pad="34"/>
 <wire x1="9.7" y1="26.785" x2="6.535" y2="26.785" width="0.3048" layer="1"/>
@@
 <contactref element="D1" pad="A"/>
 <contactref element="U$2" pad="P+"/>
-<wire x1="13.36" y1="2.54" x2="14.7" y2="3.88" width="1.016" layer="1"/>
-<wire x1="14.7" y1="3.88" x2="14.7" y2="8.89" width="1.016" layer="1"/>
+<wire x1="15.9" y1="2.54" x2="14.7" y2="8.89" width="0" layer="19" extent="1-1"/>
 </signal>
 <signal name="N$40">
@@
 <wire x1="18.025" y1="23.035" x2="14.95" y2="23.035" width="0.3048" layer="1"/>
 </signal>
-<signal name="+3V3">
-<contactref element="C5" pad="1"/>
-<contactref element="U$4" pad="40"/>
+<signal name="N$37">
+<via x="32.385" y="4.445" extent="1-16" drill="1.4"/>
+</signal>
+<signal name="N$38">
+<contactref element="U$4" pad="15"/>
+<contactref element="L2" pad="2"/>
+<wire x1="25.4" y1="8.85" x2="15.7" y2="25.785" width="0" layer="19" extent="1-1"/>
+</signal>
+<signal name="N$42">
+<contactref element="L2" pad="1"/>
+<contactref element="R3" pad="2"/>
+<contactref element="U$4" pad="12"/>
+<wire x1="19.265" y1="9.525" x2="15.7" y2="24.285" width="0" layer="19" extent="1-1"/>
+<wire x1="25.4" y1="3.85" x2="19.265" y2="9.525" width="0" layer="19" extent="1-1"/>
+</signal>
+<signal name="N$41">
+<contactref element="U$4" pad="11"/>
+<contactref element="R4" pad="2"/>
+<contactref element="R5" pad="2"/>
+<wire x1="18.2" y1="19.05" x2="15.7" y2="23.785" width="0" layer="19" extent="1-1"/>
+<wire x1="16.93" y1="15.875" x2="18.2" y2="19.05" width="0" layer="19" extent="1-1"/>
+</signal>
+<signal name="VDD1">
 <contactref element="R2" pad="2"/>
 <contactref element="C10" pad="1"/>
-<contactref element="U$4" pad="11"/>
 <contactref element="U$4" pad="19"/>
-<contactref element="U$4" pad="30"/>
-<contactref element="C6" pad="1"/>
-<wire x1="10.45" y1="29.035" x2="10.45" y2="29.809" width="0.3048" layer="1"/>
-<wire x1="10.45" y1="29.809" x2="10.16" y2="30.099" width="0.3048" layer="1"/>
-<wire x1="8.089" y1="30.099" x2="7.2" y2="29.21" width="0.3048" layer="1"/>
-<wire x1="10.16" y1="30.099" x2="8.089" y2="30.099" width="0.3048" layer="1"/>
-<wire x1="7.2" y1="21.59" x2="9.395" y2="23.785" width="0.3048" layer="1"/>
-<wire x1="9.395" y1="23.785" x2="9.7" y2="23.785" width="0.3048" layer="1"/>
+<contactref element="VD2" pad="A"/>
 <wire x1="15.7" y1="27.785" x2="16.665" y2="27.785" width="0.3048" layer="1"/>
 <wire x1="16.665" y1="27.785" x2="17.145" y2="27.305" width="0.3048" layer="1"/>
@@
 <wire x1="18.2" y1="26.035" x2="18.2" y2="27.266" width="0.3048" layer="1"/>
 <wire x1="18.2" y1="27.266" x2="18.161" y2="27.305" width="0.3048" layer="1"/>
-<via x="1.905" y="4.445" extent="1-16" drill="1.4"/>
-<wire x1="15.7" y1="23.785" x2="18.2" y2="26.035" width="0" layer="19" extent="1-1"/>
+<contactref element="C5" pad="1"/>
+<contactref element="U$4" pad="40"/>
+<wire x1="7.2" y1="21.59" x2="9.395" y2="23.785" width="0.3048" layer="1"/>
+<wire x1="9.395" y1="23.785" x2="9.7" y2="23.785" width="0.3048" layer="1"/>
+<via x="3.81" y="20.32" extent="1-16" drill="0.35"/>
+<wire x1="3.81" y1="20.32" x2="7.112" y2="20.32" width="0.3048" layer="16"/>
+<via x="7.112" y="20.32" extent="1-16" drill="0.35"/>
+<wire x1="7.112" y1="20.32" x2="7.2" y2="20.408" width="0.3048" layer="1"/>
+<wire x1="7.2" y1="20.408" x2="7.2" y2="21.59" width="0.3048" layer="1"/>
+<contactref element="U$4" pad="30"/>
+<contactref element="C6" pad="1"/>
+<wire x1="10.45" y1="29.035" x2="10.45" y2="29.809" width="0.3048" layer="1"/>
+<wire x1="10.45" y1="29.809" x2="10.16" y2="30.099" width="0.3048" layer="1"/>
+<wire x1="8.089" y1="30.099" x2="7.2" y2="29.21" width="0.3048" layer="1"/>
+<wire x1="10.16" y1="30.099" x2="8.089" y2="30.099" width="0.3048" layer="1"/>
 <wire x1="10.45" y1="29.035" x2="15.7" y2="27.785" width="0" layer="19" extent="1-1"/>
 <wire x1="9.7" y1="23.785" x2="10.45" y2="29.035" width="0" layer="19" extent="1-1"/>
-<wire x1="1.905" y1="4.445" x2="7.2" y2="21.59" width="0" layer="19" extent="1-1"/>
-</signal>
-<signal name="N$37">
-<via x="32.385" y="4.445" extent="1-16" drill="1.4"/>
+<wire x1="5.08" y1="5.842" x2="3.81" y2="20.32" width="0" layer="19" extent="1-1"/>
+</signal>
+<signal name="+5V">
+<contactref element="VD1" pad="C"/>
+<via x="1.905" y="1.905" extent="1-16" drill="1.4"/>
+<wire x1="1.905" y1="1.905" x2="17.653" y2="6.985" width="0" layer="19" extent="1-1"/>
+</signal>
+<signal name="+3V3">
+<contactref element="VD2" pad="C"/>
+<via x="1.905" y="4.445" extent="1-16" drill="1.4"/>
+<wire x1="1.905" y1="4.445" x2="5.08" y2="4.318" width="0" layer="19" extent="1-1"/>
 </signal>
 </signals>

Commit message: updates
Parts:
- renumbered U$4 to NCN5120
Routing:
- net GND: track 79.3 -> 126.9 mm, vias 1 -> 4
- net VDD1: track 19.4 -> 58.8 mm, vias 2 -> 4
- net N$42: track 0.00 -> 26.8 mm, vias 0 -> 2
- net VDD2: track 0.00 -> 25.3 mm, vias 0 -> 2
- net N$38: track 0.00 -> 22.9 mm, vias 0 -> 2
- net +5V: track 0.00 -> 17.9 mm, vias 1 -> 2
- net N$222: track 0.00 -> 12.5 mm, vias 0 -> 2
- net N$41: track 0.00 -> 12.5 mm, vias 0 -> 2
- net N$174: track 0.00 -> 8.40 mm, vias 0 -> 2
- net N$203: track 0.00 -> 6.85 mm
- net N$140: track 2.04 -> 8.67 mm, vias 1 -> 2
- net N$9: track 12.8 -> 19.3 mm, vias 0 -> 2
- net TXD: track 0.00 -> 5.95 mm, vias 0 -> 2
- net RXD: track 0.00 -> 3.40 mm, vias 0 -> 1
- net +3V3: track 0.00 -> 3.23 mm
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- added copper zone on layer 1, net GND
- added copper zone on layer 1, net N$9
Other:
- board text added: "(SCL) PA23"
- board text added: "(SDA) PA22"
- board text added: "Konnektduino KNX Rev 1.0 0xCDDC"
- board text added: "PA10 (TX)"
- board text added: "PA11 (RX)"
- board text removed: "PA10"
- board text removed: "PA11"
- board text removed: "PA22"
- board text removed: "PA23"
