File: eagle/Konnektduino.knx.Rev.1.0.sch (EAGLE design)
At the start: 18 parts, among them Y2 16MHz

Commit message: updates
Parts:
- removed JP5: (no value), pinhead:PINHD-1X1
- added C11: 10uF, rcl:C-EUC0603
- added L2: 220uH, Wuerth_PowerMagnetics:WE-PD2_7850
- added R3: 1, rcl:R-EU_R0603
- added R4: 33k, rcl:R-EU_R0603
- added R5: 180k, rcl:R-EU_R0603
- added VD1, VD2: (no value), diode:DIODE-SCHOTTKY-0603
- renumbered Y2 to Y1
Connections:
- removed net SAVEB: JP5.1, U$4.SAVEB
- new net +5V: VD1.C
- new net N$38: L2.2, U$4.VSW2
- new net N$41: R4.2, R5.2, U$4.VDD2MV
- new net N$42: L2.1, R3.2, U$4.VDD2MC
- new net VDD1: C10.1, C5.1, C6.1, R2.2, U$4.VDD, U$4.VDD1, U$4.VDDA, VD2.A
- new net VDD2: C11.1, R3.1, R4.1, U$4.VDD2, VD1.A
- net +3V3: now also VD2.C; no longer C10.1, C5.1, C6.1, R2.2, U$4.VDD, U$4.VDD1, U$4.VDD2MV, U$4.VDDA
- net GND: now also C11.2, R5.1

Commit message: updates
Parts:
- renumbered U$4 to NCN5120
